File: board/schematics/GrowMe.kicad_sch (KiCad schematic)
At the start: 21 parts, among them J1 Conn_01x02_Male, J2 Conn_01x02_Male, M1 Stepper_Motor_bipolar, M2 Stepper_Motor_bipolar, M3 Stepper_Motor_bipolar, M4 Stepper_Motor_bipolar, M5 Stepper_Motor_bipolar, M6 Stepper_Motor_bipolar, U1 ESP32-DEVKITC

Commit message: feat: update sheet layout
Parts:
- added C?: 1uF, symbol Device:C
- added C?: 10uF, symbol Device:C
- added C?: 0.1uF, symbol Device:C
- added D? (x2): 1N4001, Diode_THT:D_DO-41_SOD81_P10.16mm_Horizontal, symbol Diode:1N4001
- added J?: Power Input, symbol Connector:Screw_Terminal_01x02
- added R?: 330, symbol Device:R_US
- added R?: 560, symbol Device:R_US
- added U?: LM317_TO-220, Package_TO_SOT_THT:TO-220-3_Vertical, symbol Regulator_Linear:LM317_TO-220
Connections:
- net +12V: now also C?.1, D?.1 (K), J?.2 (Pin_2), U?.3 (VI)
- net +3V3: now also C?.1, D?.1 (K), D?.2 (A), R?.1, U?.2 (VO)
- net GND: now also J?.1 (Pin_1)
- new net: C?.1, D?.2 (A), R?.1, R?.2, U?.1 (ADJ)
- new net: C?.2, C?.2, C?.2, R?.2
Other:
- removed sheet Power
- note added: "Motor connections"
- note added: "Power input"
- note removed: "Motor Block 2"
- moved on the sheet: A1, A2, A3, A4, A5, A6, C1, C2, C3, C4, C5, C6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

Commit message: feat: update power management
Parts:
- removed C?: 1uF, symbol Device:C
- removed C?: 10uF, symbol Device:C
- removed C?: 0.1uF, symbol Device:C
- removed D? (x2): 1N4001, Diode_THT:D_DO-41_SOD81_P10.16mm_Horizontal, symbol Diode:1N4001
- removed M1, M2, M3, M4, M5, M6: Stepper_Motor_bipolar, symbol Motor:Stepper_Motor_bipolar
- removed R?: 330, symbol Device:R_US
- removed R?: 560, symbol Device:R_US
- removed U?: LM317_TO-220, Package_TO_SOT_THT:TO-220-3_Vertical, symbol Regulator_Linear:LM317_TO-220
- added C7: 10uF, symbol Device:C
- added C8: 22uF, symbol Device:C
- added J4: M1_CONN, symbol Connector:Conn_01x05_Male
- added J5: M4_CONN, symbol Connector:Conn_01x05_Male
- added J6: M2_CONN, symbol Connector:Conn_01x05_Male
- added J7: M5_CONN, symbol Connector:Conn_01x05_Male
- added J8: M3_CONN, symbol Connector:Conn_01x05_Male
- added J9: M6_CONN, symbol Connector:Conn_01x05_Male
- added U2: LM1117-3.3, symbol Regulator_Linear:LM1117-3.3
- gave numbers to parts that had none: 1
Connections:
- net +3V3: now also C8.1, U2.2 (VO)
- net GND: now also C7.2, C8.2, U2.1 (GND); no longer U1.32 (GND2)
- net at A4.4 (1A): now also J7.2 (Pin_2)
- net at A4.3 (1B): now also J7.1 (Pin_1)
- net at A4.5 (2A): now also J7.3 (Pin_3)
- net at A4.6 (2B): now also J7.4 (Pin_4)
- net at A2.4 (1A): now also J5.2 (Pin_2)
- net at A2.3 (1B): now also J5.1 (Pin_1)
- net at A2.5 (2A): now also J5.3 (Pin_3)
- net at A2.6 (2B): now also J5.4 (Pin_4)
- net at A6.3 (1B): now also J9.1 (Pin_1)
- net at A6.4 (1A): now also J9.2 (Pin_2)
- net at A6.5 (2A): now also J9.3 (Pin_3)
- net at A6.6 (2B): now also J9.4 (Pin_4)
- net at A5.3 (1B): now also J8.1 (Pin_1)
- net at A5.4 (1A): now also J8.2 (Pin_2)
- net at A5.5 (2A): now also J8.3 (Pin_3)
- net at A5.6 (2B): now also J8.4 (Pin_4)
- net at A3.4 (1A): now also J6.2 (Pin_2)
- net at A3.3 (1B): now also J6.1 (Pin_1)
- net at A3.5 (2A): now also J6.3 (Pin_3)
- net at A3.6 (2B): now also J6.4 (Pin_4)
- net at A1.3 (1B): now also J4.1 (Pin_1)
- net at A1.4 (1A): now also J4.2 (Pin_2)
- net at A1.5 (2A): now also J4.3 (Pin_3)
- net at A1.6 (2B): now also J4.4 (Pin_4)
- net +12V renamed +5V
- net +5V: now also C7.1, U2.3 (VI)
- no-connect marks 35 -> 42
Other:
- moved on the sheet: J3
